File: Hardware/PowerUnitCoolerController.sch (KiCad schematic (older format))
At the start: 23 parts, among them IC1 LM1117-5V, IC2 ATTINY25-SS, P1 Sensor, P2 Power, P3 Programmer, P4 Cooler, Q1 BC850, Q2 IRLML6402

Commit message: - Now it seems that firmware is ready - Updated doxygen documentation for firmware
Other:
- note added: "Desolder C8 before flashing, solder back before running!"
Changed lines of the file:
@@
 EESchema Schematic File Version 2
-LIBS:lm1117
 LIBS:power
 LIBS:device
@@
 LIBS:contrib
 LIBS:valves
+LIBS:lm1117
 LIBS:fossa library
 LIBS:PowerUnitCoolerController-cache
@@
 Wire Wire Line
 	7590 2620 7790 2620
+Text Notes 5750 4150 0    60   ~ 0
+Desolder C8 before flashing, solder back before running!
 $EndSCHEMATC
